File: hw/hw.kicad_sch (KiCad schematic)
At the start: 0 parts

Commit message: Issue #25: add Polyfuse_TBD project symbol and schematic updates
Other:
- added sheet step01_power (step01_power.kicad_sch)
Changed lines of the file:
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@@
 	(generator_version "9.0")
 	(paper "A4")
+	(sheet
+		(at 87.63 68.58)
+		(size 12.7 3.81)
+		(exclude_from_sim no)
+		(in_bom yes)
+		(on_board yes)
+		(dnp no)
+		(fields_autoplaced yes)
+		(stroke
+			(width 0.1524)
+			(type solid)
+		)
+		(fill
+			(color 0 0 0 0.0000)
+		)
+		(property "Sheetname" "step01_power"
+			(at 87.63 67.8684 0)
+			(effects
+				(font
+					(size 1.27 1.27)
+				)
+				(justify left bottom)
+			)
+		)
+		(property "Sheetfile" "step01_power.kicad_sch"
+			(at 87.63 72.9746 0)
+			(effects
+				(font
+					(size 1.27 1.27)
+				)
+				(justify left top)
+			)
+		)
+		(instances
+			(project "hw"
+				(path "/7b66d93d-d6d0-4bd4-83b3-6fc711e21073"
+					(page "2")
+				)
+			)
+		)
+	)
 	(sheet_instances
 		(path "/"
